File: experimentboard.brd (EAGLE design)
At the start: 110.5 x 100 mm, 182 parts, among them IC1 TL072P, IC2 LM317, IC3 LM337, IC4 TL072P, IC5 TL072P, IC6 TL072P, P1 PLR135/T9, P9 P9, Q1 BS170, Q2 BS170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

Commit message: Use CAT24C256 with named package suffix
Parts:
- U3: value CAT24C256 -> CAT24C256YI-GT3
Changed lines of the file:
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@@
 <attribute name="VALUE" x="100.9015" y="69.81825" size="1.27" layer="27" ratio="10" rot="R180"/>
 </element>
-<element name="U3" library="0000halfgaar" package="TSSOP8" value="CAT24C256" x="76.2" y="81.5975" smashed="yes">
+<element name="U3" library="0000halfgaar" package="TSSOP8" value="CAT24C256YI-GT3" x="76.2" y="81.5975" smashed="yes">
 <attribute name="NAME" x="79.6925" y="80.772" size="1.27" layer="25" ratio="10" rot="R180"/>
 <attribute name="VALUE" x="79.248" y="79.0575" size="1.27" layer="27" ratio="10" rot="R90"/>

Commit message: Changed opamp to value OPA2134
Parts:
- IC1, IC4, IC5, IC6: value TL072P -> OPA2134
Changed lines of the file:
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@@
 <attribute name="VALUE" x="71.882" y="65.4685" size="1.27" layer="27" ratio="10" rot="R270"/>
 </element>
-<element name="IC1" library="0000halfgaar" package="DIL8" value="TL072P" x="91.44" y="19.05" rot="R90"/>
+<element name="IC1" library="0000halfgaar" package="DIL8" value="OPA2134" x="91.44" y="19.05" rot="R90"/>
 <element name="1_R1" library="rcl" package="0207/7" value="7.5k" x="99.06" y="41.91" smashed="yes" rot="R270">
 <attribute name="NAME" x="98.552" y="42.8625" size="1.27" layer="25" ratio="10" rot="R270"/>
@@
 <attribute name="VALUE" x="56.896" y="79.2988" size="1.27" layer="27" ratio="10" rot="R180"/>
 </element>
-<element name="IC4" library="0000halfgaar" package="DIL8" value="TL072P" x="67.31" y="19.05" rot="R90"/>
+<element name="IC4" library="0000halfgaar" package="DIL8" value="OPA2134" x="67.31" y="19.05" rot="R90"/>
 <element name="3_R1" library="rcl" package="0207/7" value="7.5k" x="74.93" y="41.91" smashed="yes" rot="R270">
 <attribute name="NAME" x="74.26325" y="44.1325" size="1.27" layer="25" ratio="10" rot="R270"/>
@@
 <attribute name="VALUE" x="63.881" y="8.763" size="1.27" layer="27" ratio="10"/>
 </element>
-<element name="IC5" library="0000halfgaar" package="DIL8" value="TL072P" x="43.18" y="19.05" rot="R90"/>
+<element name="IC5" library="0000halfgaar" package="DIL8" value="OPA2134" x="43.18" y="19.05" rot="R90"/>
 <element name="5_R1" library="rcl" package="0207/7" value="7.5k" x="50.8" y="41.91" smashed="yes" rot="R270">
 <attribute name="NAME" x="50.292" y="43.815" size="1.27" layer="25" ratio="10" rot="R270"/>
@@
 <attribute name="VALUE" x="39.751" y="8.763" size="1.27" layer="27" ratio="10"/>
 </element>
-<element name="IC6" library="0000halfgaar" package="DIL8" value="TL072P" x="16.51" y="19.05" rot="R90"/>
+<element name="IC6" library="0000halfgaar" package="DIL8" value="OPA2134" x="16.51" y="19.05" rot="R90"/>
 <element name="7_R1" library="rcl" package="0207/7" value="7.5k" x="24.13" y="41.91" smashed="yes" rot="R270">
 <attribute name="NAME" x="23.46325" y="44.29125" size="1.27" layer="25" ratio="10" rot="R270"/>

Commit message: One more decoupling cap
Parts:
- added C17: 10 µF, rcl:E2-5
Connections:
- net DGND: now also C17.-
- net VDD_5V: now also C17.+
Routing:
- net VDD_5V: track 15.5 -> 19.6 mm
Other:
- board text added: "JP2/3 closed: feed BBB PWR"
- board text removed: "Closed: feed BBB PWR"
Changed lines of the file:
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@@
 <text x="100.965" y="55.08625" size="1.016" layer="21">24b ljust</text>
 <text x="100.965" y="53.18125" size="1.016" layer="21">24b I2S</text>
-<text x="51.27625" y="86.36" size="1.016" layer="21">Closed: feed
+<text x="55.245" y="86.36" size="1.016" layer="21">JP2/3 closed: feed
 BBB PWR</text>
 <text x="107.95" y="6.35" size="1.016" layer="21" rot="R90">Beagle Bone multi-channel audio decoder
@@
 </element>
 <element name="P9" library="0000halfgaar" package="HEADERS23-2" value="P9" x="52.07" y="93.98" smashed="yes">
-<attribute name="NAME" x="66.675" y="87.85225" size="1.27" layer="25" ratio="10"/>
+<attribute name="NAME" x="74.45375" y="88.011" size="1.27" layer="25" ratio="10"/>
 <attribute name="VALUE" x="89.535" y="87.884" size="1.27" layer="27" ratio="10"/>
 </element>
@@
 </element>
 <element name="U3" library="0000halfgaar" package="TSSOP8" value="CAT24C256YI-GT3" x="76.2" y="81.5975" smashed="yes">
-<attribute name="NAME" x="79.6925" y="80.772" size="1.27" layer="25" ratio="10" rot="R180"/>
+<attribute name="NAME" x="77.94625" y="78.07325" size="1.27" layer="25" ratio="10" rot="R180"/>
 <attribute name="VALUE" x="79.248" y="79.0575" size="1.27" layer="27" ratio="10" rot="R90"/>
 </element>
@@
 <attribute name="NAME" x="6.82625" y="0.635" size="1.016" layer="25" ratio="10"/>
 <attribute name="VALUE" x="10.795" y="-1.905" size="1.016" layer="27" ratio="10"/>
+</element>
+<element name="C17" library="rcl" package="E2-5" value="10 µF" x="52.07" y="86.36" smashed="yes">
+<attribute name="NAME" x="53.81625" y="83.2485" size="1.27" layer="25" ratio="10"/>
+<attribute name="VALUE" x="54.61" y="84.201" size="1.27" layer="27" ratio="10"/>
 </element>
 </elements>
@@
 <contactref element="Q1" pad="S"/>
 <contactref element="Q2" pad="S"/>
+<contactref element="C17" pad="-"/>
 </signal>
 <signal name="AGND">
@@
 <wire x1="52.07" y1="95.25" x2="52.07" y2="92.71" width="1.016" layer="1"/>
 <wire x1="45.72" y1="83.82" x2="46.99" y2="85.09" width="0.8128" layer="1"/>
-<wire x1="46.99" y1="85.09" x2="46.99" y2="88.9" width="0.8128" layer="1"/>
+<wire x1="46.99" y1="85.09" x2="46.99" y2="86.36" width="0.8128" layer="1"/>
+<wire x1="46.99" y1="86.36" x2="46.99" y2="88.9" width="0.8128" layer="1"/>
 <wire x1="46.99" y1="88.9" x2="48.26" y2="90.17" width="0.8128" layer="1"/>
 <wire x1="48.26" y1="90.17" x2="50.8" y2="90.17" width="0.8128" layer="1"/>
 <wire x1="50.8" y1="90.17" x2="52.07" y2="91.44" width="0.8128" layer="1"/>
 <wire x1="52.07" y1="91.44" x2="52.07" y2="92.71" width="0.8128" layer="1"/>
+<contactref element="C17" pad="+"/>
+<wire x1="51.054" y1="86.36" x2="46.99" y2="86.36" width="0.8128" layer="1"/>
 </signal>
 <signal name="N$4">
